File: Universal JAMMA Interface.kicad_pcb (KiCad board)
At the start: 2 copper layers, 111 x 60.8 mm, 31 parts, among them U1 LM386, U2 DIP-14_W7.62mm_Socket

Commit message: add +12V
Parts:
- moved -5V 2.00 mm to (190.0, 86.8)
Connections:
- POWER pad 3: -5V -> +12V
Routing:
- net +12V: track 54.7 -> 59.8 mm
- net -5V: track 48.8 -> 49.8 mm

Commit message: redesign
Parts:
- AUDIO: value PinHeader_1x02_P2.54mm_Vertical -> PinHeader_1x03_P2.54mm_Vertical; footprint Connector_PinHeader_2.54mm:PinHeader_1x02_P2.54mm_Vertical -> Connector_PinHeader_2.54mm:PinHeader_1x03_P2.54mm_Vertical
- POWER: value PinHeader_1x08_P2.54mm_Vertical -> PinHeader_1x09_P2.54mm_Vertical; footprint Connector_PinHeader_2.54mm:PinHeader_1x08_P2.54mm_Vertical -> Connector_PinHeader_2.54mm:PinHeader_1x09_P2.54mm_Vertical
- moved DIRECTIONALS 21.3 mm to (99.0, 96.0)
- moved AUDIO 10.3 mm to (132.0, 92.5)
- moved MODE 6.88 mm to (142.5, 92.5)
- moved SVC 6.00 mm to (155.5, 92.5)
- moved VIDEO 5.06 mm to (163.5, 92.5)
- moved POWER 4.00 mm to (179.0, 92.5)
- moved +5V 2.82 mm to (195.0, 86.8)
- moved CONTROLS 2.61 mm to (99.0, 90.0)
- moved VOLUME 2.00 mm to (111.0, 107.5)
- moved -5V 0.75 mm to (189.2, 86.8)
- renumbered SWITCHES to CONTROLS, CONTROLS to DIRECTIONALS
Connections:
- POWER pad 5: +5V -> -5V
Routing:
- net GND: track 691.2 -> 746.4 mm
- net 2P_R: track 24.8 -> 45.6 mm
- net 2P_L: track 25.4 -> 44.4 mm
- net 2P_D: track 26.0 -> 43.8 mm
- net 2P_U: track 26.6 -> 43.2 mm
- net 1P_U: track 24.2 -> 34.6 mm
- net 1P_D: track 24.8 -> 34.0 mm
- net 1P_L: track 25.3 -> 34.5 mm
- net 1P_R: track 25.9 -> 35.1 mm
- net TEST: track 61.0 -> 65.7 mm
- net PREAMP: track 45.5 -> 41.1 mm
- net AUDIO_R: track 27.1 -> 22.7 mm
- net AUDIO_L: track 27.0 -> 22.8 mm
- net -5V: track 49.8 -> 53.9 mm
- net +5V: track 187.6 -> 191.6 mm
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Other:
- board text added: "RET"
- board text removed: "(+) SPKR"
- board text removed: "(-) GND"
- board text removed: "(-) VID GND"
- board text removed: "1P BUTTON 1"
- board text removed: "1P BUTTON 2"
- board text removed: "1P BUTTON 3"
- board text removed: "1P BUTTON 4"
- board text removed: "1P DOWN"
- board text removed: "1P LEFT"
- board text removed: "1P RIGHT"
- board text removed: "1P UP"
- board text removed: "2P BUTTON 1"
- board text removed: "2P BUTTON 2"
- board text removed: "2P BUTTON 3"
- board text removed: "2P BUTTON 4"
- board text removed: "2P DOWN"
- board text removed: "2P LEFT"
- board text removed: "2P RIGHT"
- board text removed: "2P UP"
- board text removed: "CNTR 1"
- board text removed: "CNTR 2"
- board text removed: "COIN 1 SW"
- board text removed: "COIN 2 SW"
- board text removed: "GND (-)"
- board text removed: "LOCKOUT 1"
- board text removed: "LOCKOUT 2"
- board text removed: "SERVICE SW"
- board text removed: "SPKR (-)"
- board text removed: "TEST SW"
- board text removed: "TILT SW"
- board text removed: "VID BLUE"
- board text removed: "VID CSYNC"
- board text removed: "VID GRN"
- board text removed: "VID RED"
