File: Universal JAMMA Microcontroller.kicad_pcb (KiCad board)
At the start: 2 copper layers, 111 x 78.8 mm, 43 parts, among them U1 LM386, U2 74LS86, U3 MC34063AP, U4 328P

Commit message: Minor tweaks
Other:
- board text added: "UNIVERSAL JAMMA MICROCONTROLLER INTERFACE"
- board text removed: "UNIVERSAL JAMMA MICROCONTROLLER"
Changed lines of the file:
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@@
 		)
 	)
-	(gr_text "UNIVERSAL JAMMA MICROCONTROLLER"
+	(gr_text "UNIVERSAL JAMMA MICROCONTROLLER INTERFACE"
 		(at 149.457988 78.8 0)
 		(layer "F.SilkS")
@@
 	)
 	(gr_text "SYNC COMBINER"
-		(at 178.565357 119.176679 0)
-		(layer "F.SilkS")
-		(effects
+		(at 178.089166 119.176679 0)
+		(layer "F.SilkS")
+		(effects
