File: Williams JAMMA Interface.kicad_pcb (KiCad board)
At the start: 2 copper layers, 111 x 74.8 mm, 41 parts, among them P1 10K, U1 LM386, U2 DIP-14_W7.62mm_Socket, U3 MC34063AP

Commit message: Williams System JAMMA Rev. 1
Parts:
- removed -5V: TestPoint_Pad_D1.0mm, TestPoint:TestPoint_Pad_D1.0mm
- removed the CONTROLS at (99.0, 89.2)
- removed Ground (x2): PinHeader_1x04_P2.54mm_Vertical, Connector_PinHeader_2.54mm:PinHeader_1x04_P2.54mm_Vertical
- added CONTROLS: PinHeader_1x12_P2.54mm_Vertical, Connector_PinHeader_2.54mm:PinHeader_1x12_P2.54mm_Vertical, F.Cu at (99.2, 85.2)
- added GND: Molex_KK-396_5273-08A_1x08_P3.96mm_Vertical, Connector_Molex:Molex_KK-396_5273-08A_1x08_P3.96mm_Vertical, F.Cu at (172.6, 128.2)
- JAMMA / CHAMMA: renamed from JAMMA
- POWER: value PinHeader_1x09_P2.54mm_Vertical -> Molex_KK-396_5273-09A_1x09_P3.96mm_Vertical; footprint Connector_PinHeader_2.54mm:PinHeader_1x09_P2.54mm_Vertical -> Connector_Molex:Molex_KK-396_5273-09A_1x09_P3.96mm_Vertical
- U3: footprint Package_DIP:DIP-8_W7.62mm_Socket_LongPads -> Package_DIP:DIP-8_W7.62mm_LongPads
- moved TEST 94.9 mm to (97.2, 134.6)
- moved -12V 16.4 mm to (157.6, 124.5)
- moved POWER 13.2 mm to (168.6, 84.4), turned to 0 degrees
- moved +5V 11.0 mm to (195.0, 75.8), turned to 180 degrees
- moved +12V 11.0 mm to (183.2, 75.8), turned to 180 degrees
- moved GND 6.84 mm to (203.8, 93.6)
- moved AUDIO 5.75 mm to (127.6, 96.2)
- moved MODE 5.67 mm to (138.2, 96.2)
- moved SVC 5.67 mm to (151.2, 96.2)
- moved VIDEO 5.67 mm to (159.2, 96.2)
- moved L1 2.30 mm to (109.2, 125.5)
- moved C8 2.20 mm to (151.8, 126.2)
- moved R7 2.10 mm to (160.4, 130.2)
- moved R8 1.80 mm to (163.2, 130.2)
- moved C6 1.80 mm to (118.2, 125.5)
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Connections:
- JAMMA / CHAMMA pad 26: (no net) -> 1P_B5
- JAMMA / CHAMMA pad 27: GND -> 1P_B6
- JAMMA / CHAMMA pad d: (no net) -> 2P_B5
- JAMMA / CHAMMA pad e: GND -> 2P_B6
Routing:
- net GND: track 839.6 -> 908.6 mm
- net TEST: track 65.7 -> 102.4 mm, vias 1 -> 4
- net 1P_B5: track 0.00 -> 23.9 mm
- net 1P_B6: track 0.00 -> 23.4 mm
- net SWE: track 47.8 -> 30.0 mm
- net 2P_B5: track 0.00 -> 16.8 mm
- net 2P_B6: track 0.00 -> 16.4 mm
- net -5V: track 48.8 -> 32.5 mm, vias 1 -> 0
- net +5V: track 336.0 -> 347.3 mm, vias 5 -> 3
- net +12V: track 61.1 -> 51.6 mm, vias 1 -> 0
- net 1P_R: track 35.1 -> 43.5 mm
- net 2P_B1: track 25.5 -> 19.3 mm
- net 2P_B2: track 24.9 -> 18.7 mm
- net 2P_B4: track 23.7 -> 17.5 mm
- net 2P_B3: track 24.3 -> 18.1 mm
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Other:
- board size 111 x 74.8 mm -> 112.2 x 74.8 mm
- board text added: "1P B5"
- board text added: "1P B6"
- board text added: "1P ST"
- board text added: "2P B5"
- board text added: "2P B6"
- board text added: "2P ST"
- board text added: "C/S"
- board text added: "JP1"
- board text added: "SYN 1"
- board text added: "SYN 2"
- board text removed: "1P START"
- board text removed: "2P START"
- board text removed: "COMP/S"
- board text removed: "GND"
- board text removed: "SYNC 1"
- board text removed: "SYNC 2"

Commit message: minor tweaks
Parts:
- moved -12V 37.7 mm to (183.6, 97.2), turned to 180 degrees
- moved GND 3.60 mm to (203.8, 97.2), turned to -90 degrees
- moved +12V 3.09 mm to (180.4, 77.2)
- moved +5V 1.87 mm to (193.8, 77.2)
- moved U2 0.53 mm to (176.6, 101.8)
- moved P1 0.40 mm to (110.2, 107.4)
- moved R3 0.28 mm to (122.4, 113.4)
- moved C1 0.21 mm to (119.8, 113.4)
- moved R1 0.20 mm to (127.8, 105.8)
- moved U1 0.20 mm to (139.2, 113.4)
- moved R2 0.15 mm to (125.2, 105.8)
Routing:
- net VID_SYN1: track 33.2 -> 34.3 mm
- net +12V: track 51.6 -> 52.5 mm
- net +5V: track 347.3 -> 348.0 mm
- net SPKR+: track 80.6 -> 81.1 mm
- net VID_NXOR_R5: track 6.84 -> 7.39 mm
