File: JAMMA Microcontroller Adapter.kicad_pcb (KiCad board)
At the start: 2 copper layers, 111 x 91.4 mm, 36 parts, among them U1 LM386, U2 74LS86, U3 MC34063AP, U4 328P

Commit message: 152 becomes 2A152J (reduced noise)
Parts:
- C8: value 152 -> 2A152J
Changed lines of the file:
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@@
 			)
 		)
-		(property "Value" "152"
+		(property "Value" "2A152J"
 			(at 2.5 0 90)
 			(layer "F.SilkS")
