File: TRON to JAMMA Adapter.kicad_pcb (KiCad board)
At the start: 2 copper layers, 112.2 x 98.7 mm, 58 parts, among them P1 1K, P2 10K, P3 1K, U1 74LS86, U2A 74LS191, U2B 74LS191, U3 NE555, U4 LM386, U5 NE555

Commit message: minor routing tweak
Routing:
- net +5V: track 510.3 -> 508.7 mm
Other:
- board text added: "LVL DN"
- board text added: "LVL UP"
- board text removed: "LEVEL DN"
- board text removed: "LEVEL UP"
Changed lines of the file:
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@@
 	)
 	(gr_line
-		(start 145 78.8)
-		(end 143.4 78.8)
+		(start 145 77.235479)
+		(end 143.4 77.235479)
 		(stroke
 			(width 0.076)
@@
 	)
 	(gr_line
-		(start 143.4 78.8)
-		(end 143.4 78.098063)
+		(start 143.4 77.235479)
+		(end 143.4 76.533542)
 		(stroke
 			(width 0.076)
@@
 	)
 	(gr_line
-		(start 150 78.8)
-		(end 148.4 78.8)
+		(start 150 77.235479)
+		(end 148.4 77.235479)
 		(stroke
 			(width 0.076)
@@
 	)
 	(gr_line
-		(start 150 78.8)
-		(end 150 78.098063)
+		(start 150 77.235479)
+		(end 150 76.533542)
 		(stroke
 			(width 0.076)
@@
 	)
 	(gr_text "DOT"
-		(at 145.581535 78.964521 0)
+		(at 145.581535 77.4 0)
 		(layer "F.SilkS")
 		(effects
@@
 		)
 	)
-	(gr_text "LEVEL DN"
-		(at 147.30175 77.142858 90)
+	(gr_text "LVL DN"
+		(at 147.30175 75.333334 90)
 		(layer "F.SilkS")
 		(effects
@@
 		)
 	)
-	(gr_text "LEVEL UP"
-		(at 144.76175 77.142858 90)
+	(gr_text "LVL UP"
+		(at 144.76175 75.333334 90)
 		(layer "F.SilkS")
 		(effects
@@
 	)
 	(gr_text "PCB Design Copyright © 2025, Jonathan Zdziarski\nAll Rights Reserved"
-		(at 90.25 87.5 270)
+		(at 90.099815 63.403962 270)
 		(layer "F.Fab")
 		(effects
@@
 	)
 	(segment
-		(start 168.5 122.75)
-		(end 127.2 122.75)
+		(start 169 122.25)
+		(end 176.108223 122.25)
 		(width 0.85)
 		(layer "B.Cu")
@@
 	)
 	(segment
-		(start 179.108223 119.25)
-		(end 183.5 119.25)
-		(width 0.85)
-		(layer "B.Cu")
-		(net 55)
-	)
-	(segment
 		(start 180.75 84)
 		(end 180.75 85.75)
@@
 	)
 	(segment
+		(start 176.108223 122.25)
+		(end 183.358223 115)
+		(width 0.85)
+		(layer "B.Cu")
+		(net 55)
+	)
+	(segment
 		(start 190.533352 57.527627)
 		(end 188.4 57.527627)
@@
 	)
 	(segment
-		(start 185 117.75)
-		(end 185 115)
-		(width 0.85)
-		(layer "B.Cu")
-		(net 55)
-	)
-	(segment
 		(start 116.237594 81.792499)
 		(end 113.262983 81.792499)
@@
 	)
 	(segment
+		(start 168.5 122.75)
+		(end 169 122.25)
+		(width 0.85)
+		(layer "B.Cu")
+		(net 55)
+	)
+	(segment
 		(start 141.629 112.851)
 		(end 135.871 112.851)
@@
 	)
 	(segment
+		(start 183.358223 115)
+		(end 185 115)
+		(width 0.85)
+		(layer "B.Cu")
+		(net 55)
+	)
+	(segment
 		(start 110.739929 103.665929)
 		(end 110.684715 103.665929)
@@
 	)
 	(segment
-		(start 169 122.25)
-		(end 176.108223 122.25)
-		(width 0.85)
-		(layer "B.Cu")
-		(net 55)
-	)
-	(segment
 		(start 188.4 57.527627)
 		(end 188.4 81.44)
@@
 	)
 	(segment
-		(start 183.5 119.25)
-		(end 185 117.75)
-		(width 0.85)
-		(layer "B.Cu")
-		(net 55)
-	)
-	(segment
 		(start 190.533352 57.527627)
 		(end 190.533352 50.933357)
@@
 	)
 	(segment
-		(start 169 122.25)
-		(end 168.5 122.75)
-		(width 0.85)
-		(layer "B.Cu")
-		(net 55)
-	)
-	(segment
 		(start 121.41232 105.60768)
 		(end 112.68168 105.60768)
@@
 	)
 	(segment
-		(start 176.108223 122.25)
-		(end 179.108223 119.25)
-		(width 0.85)
-		(layer "B.Cu")
-		(net 55)
-	)
-	(segment
 		(start 180.75 85.75)
 		(end 189.56 94.56)
@@
 		(layer "B.Cu")
 		(net 55)
+	)
+	(segment
+		(start 127.2 122.75)
+		(end 168.5 122.75)
+		(width 0.85)
+		(layer "B.Cu")
+		(net 55)
