File: Blasteroids JAMMA Adapter.kicad_pcb (KiCad board)
At the start: 2 copper layers, 112.2 x 82 mm, 49 parts, among them P1 10K, U1 74LS86, U2 NE555, U3 MC34063AP, U4 LM386, U5 NE555

Commit message: minor cleanup
Parts:
- moved C12 0.10 mm to (174.8, 113.0)
Connections:
- C12 pad 1: U5_THR -> GND
- C12 pad 2: GND -> U5_THR
- JSPKR pad 2: GND -> AUDIO_R
- JSPKR pad 3: AUDIO_R -> AUDIO_L
- JSPKR pad 4: AUDIO_L -> GND
Routing:
- net GND: track 774.9 -> 797.8 mm
- net AUDIO_L: track 39.4 -> 37.5 mm
- net U5_THR: track 49.7 -> 48.1 mm, vias 3 -> 2
- net 2P_B2: track 34.7 -> 35.8 mm
- net AUDIO_R: track 38.4 -> 37.4 mm
- net VCLK2_DELAYED: track 33.9 -> 34.4 mm, vias 2 -> 1
Other:
- board text added: "SND 1"
- board text added: "SND 2"
- board text removed: "SND L"
- board text removed: "SND R"
