File: CAD/Outrun JAMMA Adapter.kicad_pcb (KiCad board)
At the start: 2 copper layers, 111 x 86.6 mm, 31 parts, among them U1 LM386, U2 MCP4902, U3 ATMEGA328

Commit message: R3 -> 2.2K
Parts:
- R3: value 10R -> 2K2
Changed lines of the file:
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@@
 			)
 		)
-		(property "Value" "10R"
+		(property "Value" "2K2"
 			(at 3.81 0 90)
 			(layer "F.SilkS")

Commit message: Switch D and G IDC connectors to prevent chafing
Parts:
- moved D 13.3 mm to (138.0, 131.2)
- moved G 12.7 mm to (119.0, 143.9)
Routing:
- net REFB: track 107.4 -> 47.4 mm, vias 1 -> 0
- net REFA: track 113.4 -> 55.5 mm
- net +5V: track 368.1 -> 390.9 mm
- net ACCEL: track 67.6 -> 56.8 mm, vias 0 -> 1
- net STEER: track 65.2 -> 54.9 mm
- net COIN_1: track 149.8 -> 159.9 mm
- net SHIFT: track 30.3 -> 40.3 mm
- net 1P_START: track 145.1 -> 154.6 mm
- net BRK: track 60.6 -> 52.1 mm, vias 1 -> 0
- net SERVICE: track 144.1 -> 149.7 mm
- net TEST: track 143.3 -> 148.6 mm
- net PB1: track 85.9 -> 85.8 mm, vias 4 -> 2
