File: CAD/Spy Hunter JAMMA Adapter.kicad_pcb (KiCad board)
At the start: 2 copper layers, 112.3 x 135.4 mm, 88 parts, among them P1 1K, P2 1K, P3 10K, P4 1K, SW2 SW_DIP_SPSTx02_Slide_9.78x7.2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, U1 74LS86, U10 NE555, U11 LM386, U12 CD4099B, U2 74LS74, U3 74LS00, U4 74LS00, U5 74LS191, U6 74LS191, U7 NE555, U8 74LS157, U9 74LS157

Commit message: Spy Hunter Rev. 1.1 (Under Development, Untested)
Parts:
- added C13: 10 uF, CP_Radial_D5.0mm_P2.00mm, F.Cu at (126.0, 82.0)
- added R13: R_Axial_DIN0204_L3.6mm_D1.6mm_P7.62mm_Horizontal, R_Axial_DIN0204_L3.6mm_D1.6mm_P7.62mm_Horizontal, F.Cu at (139.6, 43.8)
- R9: value 22R -> 2K2
- moved C9 3.74 mm to (135.8, 82.0)
- moved C1 3.44 mm to (143.4, 127.2), turned to 90 degrees
Connections:
- U11 pad 3: AUDIO_PREAMP -> AUDIO_PREAMP_COUPLED
Routing:
- net AUDIO_PREAMP_COUPLED: track 0.00 -> 47.1 mm, vias 0 -> 3
- net GND: track 1351.4 -> 1365.2 mm, vias 25 -> 27
- net AUDIO_PREAMP: track 24.2 -> 35.7 mm, vias 0 -> 3
- net U7_TRIG: track 36.3 -> 33.6 mm
Other:
- board text added: "Bally/Midway MCR III JAMMA Interface for Spy Hunter®, Rev. 1.1"
- board text removed: "Bally/Midway MCR III JAMMA Interface for Spy Hunter®, Rev. 1"

Commit message: Put component values on silkscreen R12/R13
Parts:
- R12: value R_Axial_DIN0204_L3.6mm_D1.6mm_P7.62mm_Horizontal -> 10R
- R13: value R_Axial_DIN0204_L3.6mm_D1.6mm_P7.62mm_Horizontal -> 47K

Commit message: Fix dupe of C13, rename second one to C20
Parts:
- renumbered C13 to C20
Changed lines of the file:
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@@
 		(descr "CP, Radial series, Radial, pin pitch=2.00mm, diameter=5mm, height=7mm, Electrolytic Capacitor")
 		(tags "CP Radial series Radial pin pitch 2.00mm diameter 5mm height 7mm Electrolytic Capacitor")
-		(property "Reference" "C13"
+		(property "Reference" "C20"
 			(at 0.9 -3.7 90)
 			(layer "F.SilkS")
