File: CAD/RoadBlasters JAMMA Adapter.kicad_pcb (KiCad board)
At the start: 2 copper layers, 112.2 x 82 mm, 46 parts, among them J101 Molex_KK-396_5273-10A_1x10_P3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, J102 Molex_KK-254_AE-6410-02A_1x02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, J103 Molex_KK-254_AE-6410-02A_1x02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, J104 Molex_KK-254_AE-6410-02A_1x02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, J105 Molex_KK-254_AE-6410-04A_1x04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, J106 Molex_KK-254_AE-6410-02A_1x02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, J108 Molex_KK-254_AE-6410-05A_1x05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, P1 10K, U1 74LS86, U2 NE555, U3 MC34063AP, U4 LM386

Commit message: R3 can be 2K2 for better log trim
Parts:
- R3: value 22R -> 2K2
