File: CAD/TRON to JAMMA Adapter.kicad_pcb (KiCad board)
At the start: 2 copper layers, 112.2 x 98.7 mm, 58 parts, among them P1 1K, P2 10K, P3 1K, U1 74LS86, U2A 74LS191, U2B 74LS191, U3 NE555, U4 LM386, U5 NE555

Commit message: trim shunt -> 2K2
Parts:
- R1: value R1 -> 470R
- R3: value 22R -> 2K2
- R4: value R_Axial_DIN0204_L3.6mm_D1.6mm_P7.62mm_Horizontal -> 10R
