File: CAD/Atari JAMMA Interface.kicad_pcb (KiCad board)
At the start: 2 copper layers, 112.2 x 74.8 mm, 45 parts, among them P1 10K, U1 LM386, U2 DIP-14_W7.62mm, U3 MC34063AP, U4 74LS04

Commit message: R3 audio taper, 22R -> 2.2K
Parts:
- R3: value 22R -> 2.2K
